File: hardware/kicad/hue-simple-switch-mains-panel.kicad_pcb (KiCad board)
At the start: 2 copper layers, 144 x 71 mm, 139 parts, among them J1 MAINS L/N, J2 D0 D1 D2 D3, J3 D4 D5 GND, U1 XIAO ESP32-C6

Commit message: Panel: side tabs between the boards and to the frame
Each board was held only by four tabs on its round ends. Add a tab on
each straight side at y = -3 mm (between J1 and J2 on the right, clear of
the XIAO pads on the left), tying neighbours together and the outer boards
to the side frame, so the row stays stiff while the through-hole parts are
inserted and soldered. Mouse bites on every board edge; panel DRC clean.

Co-Authored-By: Claude Opus 5.5 <noreply@anthropic.com>
Parts:
- added MB49: , , F.Cu at (84.9, 95.5)
- added MB50: , , F.Cu at (84.9, 96.5)
- added MB51: , , F.Cu at (84.9, 97.5)
- added MB52: , , F.Cu at (84.9, 98.5)
- added MB53: , , F.Cu at (127.1, 95.5)
- added MB54: , , F.Cu at (127.1, 96.5)
- added MB55: , , F.Cu at (127.1, 97.5)
- added MB56: , , F.Cu at (127.1, 98.5)
- added MB57: , , F.Cu at (128.9, 95.5)
- added MB58: , , F.Cu at (128.9, 96.5)
- added MB59: , , F.Cu at (128.9, 97.5)
- added MB60: , , F.Cu at (128.9, 98.5)
- added MB61: , , F.Cu at (171.1, 95.5)
- added MB62: , , F.Cu at (171.1, 96.5)
- added MB63: , , F.Cu at (171.1, 97.5)
- added MB64: , , F.Cu at (171.1, 98.5)
- added MB65: , , F.Cu at (172.9, 95.5)
- added MB66: , , F.Cu at (172.9, 96.5)
- added MB67: , , F.Cu at (172.9, 97.5)
- added MB68: , , F.Cu at (172.9, 98.5)
- added MB69: , , F.Cu at (215.1, 95.5)
- added MB70: , , F.Cu at (215.1, 96.5)
- added MB71: , , F.Cu at (215.1, 97.5)
- added MB72: , , F.Cu at (215.1, 98.5)
Other:
- outline, holes or cut-outs redrawn
