File: hardware/kicad/hue-simple-switch-mains.kicad_pcb (KiCad board)
At the start: 2 copper layers, 42 x 52 mm, 28 parts, among them J1 MAINS L/N, J2 D0 D1 D2 D3, J3 D4 D5 GND, U1 XIAO ESP32-C6

Commit message: Check every mains-board footprint against its datasheet (#29)
RV1 used a 1210 resistor footprint (3.2 x 2.5 mm), but the TDK SIOV
CU3225K275G2 is 8.0 x 6.3 x 4.5 mm ("3225" is in hundredths of an inch);
LCSC's package label was wrong. Other parts differed from their makers'
drawings too.

- New datasheet footprints in hardware/scripts/footprints.py:
  RV1 on TDK's land pattern (3.5 x 2.8 pads, 4.5 gap); PS1 on Hi-Link's
  drawing (rows 29.4, DC pins 15.4 apart, 1.3 drills for Ø0.8 ±0.2 pins);
  J1 KF128-5.08 (1.4 holes, 10.7 deep); J2 XY350V-3.5-4P and J3
  KF350-3.5-3P (6.9 deep). Box 3D models at datasheet size for those,
  the XIAO and the fuse, so the STEP heights are real.
- RV1 moved above the module's AC pins; J1 moved in so its real body
  clears the enclosure wall.
- N and fused L rerouted: L to N now >= 2.5 mm everywhere (was 1.76 mm
  at the fuse); mains to low voltage still >= 6 mm.
- Enclosure wire holes at the real opening heights; floor holes over
  the terminal screws.
- ERC 0, DRC 0 errors with schematic parity. Fab outputs regenerated.

Co-authored-by: Claude Opus 5.5 <noreply@anthropic.com>
Parts:
- J1: footprint TerminalBlock_Phoenix:TerminalBlock_Phoenix_MKDS-1,5-2-5.08_1x02_P5.08mm_Horizontal -> hue:TerminalBlock_Kefa_KF128-5.08_1x02
- J2: footprint TerminalBlock_Phoenix:TerminalBlock_Phoenix_PT-1,5-4-3.5-H_1x04_P3.50mm_Horizontal -> hue:TerminalBlock_Xinlaiya_XY350V-3.5_1x04
- J3: footprint TerminalBlock_Phoenix:TerminalBlock_Phoenix_PT-1,5-3-3.5-H_1x03_P3.50mm_Horizontal -> hue:TerminalBlock_Kefa_KF350-3.5_1x03
- PS1: footprint Converter_ACDC:Converter_ACDC_Hi-Link_HLK-PMxx -> hue:HiLink_HLK-PM01
- RV1: footprint Resistor_SMD:R_1210_3225Metric -> hue:RV_TDK_SIOV_CU3225
- moved RV1 2.12 mm to (92.0, 80.5)
- moved J1 0.51 mm to (115.9, 87.3)
- moved PS1 0.16 mm to (88.0, 85.3)
- moved J3 0.05 mm to (111.4, 117.5)
Routing:
- net AC_N: track 43.9 -> 33.7 mm
- net AC_L: track 24.0 -> 25.2 mm

Commit message: Add a 3-board JLCPCB assembly panel, one-sided SMD, centred CPL
- R11-R16 move to the XIAO side, so every SMD part is on one side (no
  second stencil or double-sided assembly). Each input row is now
  pull-up, 1k, 10nF; the 10nF sits at the terminal side of the 1k.
- build_panel.py: three boards on a 144 x 71 mm frame (over JLCPCB's
  70 x 70 minimum, so no extra rails), routed tabs with mouse bites,
  three fiducials, four tooling holes. Order 5 panels = 15 boards.
  Panel DRC runs in build_all; mouse bites keep >= 1 mm from mains.
- CPL written from the board: each part at its pad centre, not the
  footprint origin (KiCad puts through-hole origins on pin 1, which put
  PS1 15 mm and J2 5 mm off in JLCPCB's preview). Panel BOM/CPL use
  per-board designators (R1_1 ...) and leave out the XIAO.
- README: ordering on the panel, and which parts to check in the
  preview (D1, PS1, J1-J3).

Co-Authored-By: Claude Opus 5.5 <noreply@anthropic.com>
Parts:
- R11, R12, R13, R14, R15, R16: moved to F.Cu
- moved C11 3.60 mm to (109.4, 99.5)
- moved C12 3.60 mm to (109.4, 102.1)
- moved C13 3.60 mm to (109.4, 104.7)
- moved C14 3.60 mm to (109.4, 107.3)
- moved C15 3.60 mm to (109.4, 109.9)
- moved C16 3.60 mm to (109.4, 112.5)
- moved R11 0.20 mm to (105.8, 99.5)
- moved R12 0.20 mm to (105.8, 102.1)
- moved R13 0.20 mm to (105.8, 104.7)
- moved R14 0.20 mm to (105.8, 107.3)
- moved R15 0.20 mm to (105.8, 109.9)
- moved R16 0.20 mm to (105.8, 112.5)
Connections:
- C11 pad 1: D0 -> IN_D0
- C12 pad 1: D1 -> IN_D1
- C13 pad 1: D2 -> IN_D2
- C14 pad 1: D3 -> IN_D3
- C15 pad 1: D4 -> IN_D4
- C16 pad 1: D5 -> IN_D5
Routing:
- net IN_D5: track 5.69 -> 7.08 mm, vias 0 -> 1
- net IN_D4: track 11.3 -> 12.5 mm, vias 0 -> 1
- net IN_D3: track 10.8 -> 12.0 mm, vias 0 -> 1
- net IN_D2: track 10.4 -> 11.7 mm, vias 0 -> 1
- net IN_D1: track 10.1 -> 11.3 mm, vias 0 -> 1
- net IN_D0: track 9.70 -> 10.9 mm, vias 0 -> 1
- net D5: track 14.5 -> 13.3 mm
- net D4: track 19.7 -> 18.4 mm
- net D3: track 24.8 -> 23.6 mm
- net D2: track 29.9 -> 28.7 mm
- net D1: track 35.1 -> 33.9 mm
- net D0: track 40.2 -> 39.0 mm
