File: hardware/kicad/hue-simple-switch-mains.kicad_sch (KiCad schematic)
At the start: 28 parts, among them J1 MAINS L/N, J2 D0 D1 D2 D3, J3 D4 D5 GND, U1 XIAO ESP32-C6

Commit message: Use one 4-way block for J2 (XY350V-3.5-4P)
The BOM listed J2 as two KF350-3.5-2P blocks with quantity 1, so an order
from it came one block short. Use a single 4-way 3.5 mm side-entry block
(LCSC C557656); same footprint, pitch and height.

Co-Authored-By: Claude Opus 5.5 <noreply@anthropic.com>
Parts:
- J2: LCSC C474892 x2 -> C557656; MPN KF350-3.5-2P x2, slid together (Cixi Kefa) -> XY350V-3.5-4P (Ningbo Xinlaiya)
Changed lines of the file:
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@@
     (property "Description" "" (at 256.54 165.1 0)
       (effects (font (size 1.27 1.27)) (hide yes)))
-    (property "LCSC" "C474892 x2" (at 256.54 165.1 0)
+    (property "LCSC" "C557656" (at 256.54 165.1 0)
       (effects (font (size 1.27 1.27)) (hide yes)))
-    (property "MPN" "KF350-3.5-2P x2, slid together (Cixi Kefa)" (at 256.54 165.1 0)
+    (property "MPN" "XY350V-3.5-4P (Ningbo Xinlaiya)" (at 256.54 165.1 0)
       (effects (font (size 1.27 1.27)) (hide yes)))
     (pin "1")

Commit message: Check every mains-board footprint against its datasheet (#29)
RV1 used a 1210 resistor footprint (3.2 x 2.5 mm), but the TDK SIOV
CU3225K275G2 is 8.0 x 6.3 x 4.5 mm ("3225" is in hundredths of an inch);
LCSC's package label was wrong. Other parts differed from their makers'
drawings too.

- New datasheet footprints in hardware/scripts/footprints.py:
  RV1 on TDK's land pattern (3.5 x 2.8 pads, 4.5 gap); PS1 on Hi-Link's
  drawing (rows 29.4, DC pins 15.4 apart, 1.3 drills for Ø0.8 ±0.2 pins);
  J1 KF128-5.08 (1.4 holes, 10.7 deep); J2 XY350V-3.5-4P and J3
  KF350-3.5-3P (6.9 deep). Box 3D models at datasheet size for those,
  the XIAO and the fuse, so the STEP heights are real.
- RV1 moved above the module's AC pins; J1 moved in so its real body
  clears the enclosure wall.
- N and fused L rerouted: L to N now >= 2.5 mm everywhere (was 1.76 mm
  at the fuse); mains to low voltage still >= 6 mm.
- Enclosure wire holes at the real opening heights; floor holes over
  the terminal screws.
- ERC 0, DRC 0 errors with schematic parity. Fab outputs regenerated.

Co-authored-by: Claude Opus 5.5 <noreply@anthropic.com>
Parts:
- J1: footprint TerminalBlock_Phoenix:TerminalBlock_Phoenix_MKDS-1,5-2-5.08_1x02_P5.08mm_Horizontal -> hue:TerminalBlock_Kefa_KF128-5.08_1x02
- J2: footprint TerminalBlock_Phoenix:TerminalBlock_Phoenix_PT-1,5-4-3.5-H_1x04_P3.50mm_Horizontal -> hue:TerminalBlock_Xinlaiya_XY350V-3.5_1x04
- J3: footprint TerminalBlock_Phoenix:TerminalBlock_Phoenix_PT-1,5-3-3.5-H_1x03_P3.50mm_Horizontal -> hue:TerminalBlock_Kefa_KF350-3.5_1x03
- PS1: footprint Converter_ACDC:Converter_ACDC_Hi-Link_HLK-PMxx -> hue:HiLink_HLK-PM01
- RV1: footprint Resistor_SMD:R_1210_3225Metric -> hue:RV_TDK_SIOV_CU3225; MPN TDK SIOV B72650M0271K072 (CU3225K275G2), 275 VAC, SMD 3225 -> TDK SIOV B72650M0271K072 (CU3225K275G2), 275 VAC, 8.0 x 6.3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
Changed lines of the file:
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@@
     (property "Value" "MAINS L/N" (at 30.48 55.88 0)
       (effects (font (size 1.27 1.27))))
-    (property "Footprint" "TerminalBlock_Phoenix:TerminalBlock_Phoenix_MKDS-1,5-2-5.08_1x02_P5.08mm_Horizontal" (at 30.48 58.42 0)
+    (property "Footprint" "hue:TerminalBlock_Kefa_KF128-5.08_1x02" (at 30.48 58.42 0)
       (effects (font (size 1.27 1.27)) (hide yes)))
     (property "Datasheet" "" (at 30.48 50.8 0)
@@
     (property "Value" "D0 D1 D2 D3" (at 256.54 172.72 0)
       (effects (font (size 1.27 1.27))))
-    (property "Footprint" "TerminalBlock_Phoenix:TerminalBlock_Phoenix_PT-1,5-4-3.5-H_1x04_P3.50mm_Horizontal" (at 256.54 172.72 0)
+    (property "Footprint" "hue:TerminalBlock_Xinlaiya_XY350V-3.5_1x04" (at 256.54 172.72 0)
       (effects (font (size 1.27 1.27)) (hide yes)))
     (property "Datasheet" "" (at 256.54 165.1 0)
@@
     (property "Value" "D4 D5 GND" (at 256.54 187.96 0)
       (effects (font (size 1.27 1.27))))
-    (property "Footprint" "TerminalBlock_Phoenix:TerminalBlock_Phoenix_PT-1,5-3-3.5-H_1x03_P3.50mm_Horizontal" (at 256.54 190.5 0)
+    (property "Footprint" "hue:TerminalBlock_Kefa_KF350-3.5_1x03" (at 256.54 190.5 0)
       (effects (font (size 1.27 1.27)) (hide yes)))
     (property "Datasheet" "" (at 256.54 182.88 0)
@@
     (property "Value" "HLK-PM01" (at 104.14 55.88 0)
       (effects (font (size 1.27 1.27))))
-    (property "Footprint" "Converter_ACDC:Converter_ACDC_Hi-Link_HLK-PMxx" (at 104.14 58.42 0)
+    (property "Footprint" "hue:HiLink_HLK-PM01" (at 104.14 58.42 0)
       (effects (font (size 1.27 1.27)) (hide yes)))
     (property "Datasheet" "" (at 104.14 50.8 0)
@@
     (property "Value" "275VAC" (at 73.66 57.15 0)
       (effects (font (size 1.27 1.27))))
-    (property "Footprint" "Resistor_SMD:R_1210_3225Metric" (at 71.12 63.5 0)
+    (property "Footprint" "hue:RV_TDK_SIOV_CU3225" (at 71.12 63.5 0)
       (effects (font (size 1.27 1.27)) (hide yes)))
     (property "Datasheet" "" (at 71.12 55.88 0)
@@
     (property "LCSC" "C211106" (at 71.12 55.88 0)
       (effects (font (size 1.27 1.27)) (hide yes)))
-    (property "MPN" "TDK SIOV B72650M0271K072 (CU3225K275G2), 275 VAC, SMD 3225" (at 71.12 55.88 0)
-      (effects (font (size 1.27 1.27)) (hide yes)))
-    (pin "1")
+    (property "MPN" "TDK SIOV B72650M0271K072 (CU3225K275G2), 275 VAC, 8.0 x 6.3 x 4.5 mm" (at 71.12 55.88 0)
+      (effects (font (size 1.27 1.27)) (hide yes)))
+    (pin "1")

Commit message: 3-board JLCPCB assembly panel, one-sided SMD, centred CPL (#30)
* Add a 3-board JLCPCB assembly panel, one-sided SMD, centred CPL

- R11-R16 move to the XIAO side, so every SMD part is on one side (no
  second stencil or double-sided assembly). Each input row is now
  pull-up, 1k, 10nF; the 10nF sits at the terminal side of the 1k.
- build_panel.py: three boards on a 144 x 71 mm frame (over JLCPCB's
  70 x 70 minimum, so no extra rails), routed tabs with mouse bites,
  three fiducials, four tooling holes. Order 5 panels = 15 boards.
  Panel DRC runs in build_all; mouse bites keep >= 1 mm from mains.
- CPL written from the board: each part at its pad centre, not the
  footprint origin (KiCad puts through-hole origins on pin 1, which put
  PS1 15 mm and J2 5 mm off in JLCPCB's preview). Panel BOM/CPL use
  per-board designators (R1_1 ...) and leave out the XIAO.
- README: ordering on the panel, and which parts to check in the
  preview (D1, PS1, J1-J3).

Co-Authored-By: Claude Opus 5.5 <noreply@anthropic.com>

* Panel: side tabs between the boards and to the frame

Each board was held only by four tabs on its round ends. Add a tab on
each straight side at y = -3 mm (between J1 and J2 on the right, clear of
the XIAO pads on the left), tying neighbours together and the outer boards
to the side frame, so the row stays stiff while the through-hole parts are
inserted and soldered. Mouse bites on every board edge; panel DRC clean.

Co-Authored-By: Claude Opus 5.5 <noreply@anthropic.com>

---------

Co-authored-by: Claude Opus 5.5 <noreply@anthropic.com>
Connections:
- net D0: no longer C11.1
- net D1: no longer C12.1
- net D2: no longer C13.1
- net D3: no longer C14.1
- net D4: no longer C15.1
- net D5: no longer C16.1
- net IN_D0: now also C11.1
- net IN_D1: now also C12.1
- net IN_D2: now also C13.1
- net IN_D3: now also C14.1
- net IN_D4: now also C15.1
- net IN_D5: now also C16.1
Other:
- note added: "Each input: 10k pull-up at the pin, 1k series, 10nF at the terminal side."
- note removed: "Each input: 10k pull-up at the pin, 1k series from the terminal, 10nF at the pin."
Changed lines of the file:
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@@
     (property "Datasheet" "" (at 127 139.7 0)
       (effects (font (size 1.27 1.27)) (hide yes)))
-    (property "Description" "with the 1k, filters noise picked up by the wall wiring" (at 127 139.7 0)
+    (property "Description" "at the terminal side of the 1k: shunts noise picked up by the wall wiring" (at 127 139.7 0)
       (effects (font (size 1.27 1.27)) (hide yes)))
     (property "LCSC" "C57112" (at 127 139.7 0)
@@
   (wire (pts (xy 127 135.89) (xy 127 133.35))
     (stroke (width 0) (type default)))
-  (global_label "D0" (shape passive) (at 127 133.35 90) (fields_autoplaced yes)
+  (global_label "IN_D0" (shape passive) (at 127 133.35 90) (fields_autoplaced yes)
     (effects (font (size 1.27 1.27)) (justify left))
     (property "Intersheetrefs" "${INTERSHEET_REFS}" (at 127 133.35 0)
@@
     (property "Datasheet" "" (at 149.86 139.7 0)
       (effects (font (size 1.27 1.27)) (hide yes)))
-    (property "Description" "with the 1k, filters noise picked up by the wall wiring" (at 149.86 139.7 0)
+    (property "Description" "at the terminal side of the 1k: shunts noise picked up by the wall wiring" (at 149.86 139.7 0)
       (effects (font (size 1.27 1.27)) (hide yes)))
     (property "LCSC" "C57112" (at 149.86 139.7 0)
@@
   (wire (pts (xy 149.86 135.89) (xy 149.86 133.35))
     (stroke (width 0) (type default)))
-  (global_label "D1" (shape passive) (at 149.86 133.35 90) (fields_autoplaced yes)
+  (global_label "IN_D1" (shape passive) (at 149.86 133.35 90) (fields_autoplaced yes)
     (effects (font (size 1.27 1.27)) (justify left))
     (property "Intersheetrefs" "${INTERSHEET_REFS}" (at 149.86 133.35 0)
@@
     (property "Datasheet" "" (at 172.72 139.7 0)
       (effects (font (size 1.27 1.27)) (hide yes)))
-    (property "Description" "with the 1k, filters noise picked up by the wall wiring" (at 172.72 139.7 0)
+    (property "Description" "at the terminal side of the 1k: shunts noise picked up by the wall wiring" (at 172.72 139.7 0)
       (effects (font (size 1.27 1.27)) (hide yes)))
     (property "LCSC" "C57112" (at 172.72 139.7 0)
@@
   (wire (pts (xy 172.72 135.89) (xy 172.72 133.35))
     (stroke (width 0) (type default)))
-  (global_label "D2" (shape passive) (at 172.72 133.35 90) (fields_autoplaced yes)
+  (global_label "IN_D2" (shape passive) (at 172.72 133.35 90) (fields_autoplaced yes)
     (effects (font (size 1.27 1.27)) (justify left))
     (property "Intersheetrefs" "${INTERSHEET_REFS}" (at 172.72 133.35 0)
@@
     (property "Datasheet" "" (at 195.58 139.7 0)
       (effects (font (size 1.27 1.27)) (hide yes)))
-    (property "Description" "with the 1k, filters noise picked up by the wall wiring" (at 195.58 139.7 0)
+    (property "Description" "at the terminal side of the 1k: shunts noise picked up by the wall wiring" (at 195.58 139.7 0)
       (effects (font (size 1.27 1.27)) (hide yes)))
     (property "LCSC" "C57112" (at 195.58 139.7 0)
@@
   (wire (pts (xy 195.58 135.89) (xy 195.58 133.35))
     (stroke (width 0) (type default)))
-  (global_label "D3" (shape passive) (at 195.58 133.35 90) (fields_autoplaced yes)
+  (global_label "IN_D3" (shape passive) (at 195.58 133.35 90) (fields_autoplaced yes)
     (effects (font (size 1.27 1.27)) (justify left))
     (property "Intersheetrefs" "${INTERSHEET_REFS}" (at 195.58 133.35 0)
@@
     (property "Datasheet" "" (at 218.44 139.7 0)
       (effects (font (size 1.27 1.27)) (hide yes)))
-    (property "Description" "with the 1k, filters noise picked up by the wall wiring" (at 218.44 139.7 0)
+    (property "Description" "at the terminal side of the 1k: shunts noise picked up by the wall wiring" (at 218.44 139.7 0)
       (effects (font (size 1.27 1.27)) (hide yes)))
     (property "LCSC" "C57112" (at 218.44 139.7 0)
@@
   (wire (pts (xy 218.44 135.89) (xy 218.44 133.35))
     (stroke (width 0) (type default)))
-  (global_label "D4" (shape passive) (at 218.44 133.35 90) (fields_autoplaced yes)
+  (global_label "IN_D4" (shape passive) (at 218.44 133.35 90) (fields_autoplaced yes)
     (effects (font (size 1.27 1.27)) (justify left))
     (property "Intersheetrefs" "${INTERSHEET_REFS}" (at 218.44 133.35 0)
@@
     (property "Datasheet" "" (at 241.3 139.7 0)
       (effects (font (size 1.27 1.27)) (hide yes)))
-    (property "Description" "with the 1k, filters noise picked up by the wall wiring" (at 241.3 139.7 0)
+    (property "Description" "at the terminal side of the 1k: shunts noise picked up by the wall wiring" (at 241.3 139.7 0)
       (effects (font (size 1.27 1.27)) (hide yes)))
     (property "LCSC" "C57112" (at 241.3 139.7 0)
@@
   (wire (pts (xy 241.3 135.89) (xy 241.3 133.35))
     (stroke (width 0) (type default)))
-  (global_label "D5" (shape passive) (at 241.3 133.35 90) (fields_autoplaced yes)
+  (global_label "IN_D5" (shape passive) (at 241.3 133.35 90) (fields_autoplaced yes)
     (effects (font (size 1.27 1.27)) (justify left))
     (property "Intersheetrefs" "${INTERSHEET_REFS}" (at 241.3 133.35 0)
@@
   (text "D6-D10 unused. BOOT (GPIO9) and RESET are the buttons on the XIAO itself." (exclude_from_sim no) (at 20.32 99.06 0)
     (effects (font (size 1.27 1.27)) (justify left bottom)))
-  (text "Each input: 10k pull-up at the pin, 1k series from the terminal, 10nF at the pin." (exclude_from_sim no) (at 120.65 96.52 0)
+  (text "Each input: 10k pull-up at the pin, 1k series, 10nF at the terminal side." (exclude_from_sim no) (at 120.65 96.52 0)
     (effects (font (size 1.27 1.27)) (justify left bottom)))
   (text "Closed wall switch = pin to GND = active. Terminals are LOW VOLTAGE ONLY (3.3 V)." (exclude_from_sim no) (at 120.65 99.06 0)
