File: hardware/v2-fit/panel/v2-fit-panel.kicad_pcb (KiCad board)
At the start: 2 copper layers, 70 x 88.9 mm, 145 parts, among them J2_1 D0-D5 GND, J2_2 D0-D5 GND, J2_3 D0-D5 GND, U1_1 XIAO ESP32-C6 socket, U1_2 XIAO ESP32-C6 socket, U1_3 XIAO ESP32-C6 socket

Commit message: Hardware: v2 silkscreen in the console site's style
Label J2's contacts, draw plain references with no panel suffix, and
keep all silk clear of pads, vias and holes. Add the mains warning and
the uncertified mark on the board, so they stay once the rails are off.
The panel rails get the grid, a ruler, the setup steps and a side view.

Copper, BOM and CPL are unchanged. Local work, not approved for ordering.

Co-Authored-By: Claude Opus 5.5 <noreply@anthropic.com>
Other:
- board text added: "1"
- board text added: "2"
- board text added: "20"
- board text added: "220V AC"
- board text added: "3"
- board text added: "30"
- board text added: "40"
- board text added: "50"
- board text added: "BUILD A WALL SWITCH"
- board text added: "C1"
- board text added: "C2"
- board text added: "CHOOSE"
- board text added: "D0"
- board text added: "D1"
- board text added: "D2"
- board text added: "D3"
- board text added: "D4"
- board text added: "D5"
- board text added: "F1"
- board text added: "FOR YOUR HUE LIGHTS"
- board text added: "G"
- board text added: "HI :)"
- board text added: "HUE SWITCH"
- board text added: "HUE.TINEIRA.COM"
- board text added: "INSTALL"
- board text added: "J2"
- board text added: "MM"
- board text added: "PAIR"
- board text added: "RV1"
- board text added: "SIDE · 1:3"
- board text added: "SIMPLE · V2"
- board text added: "UNCERTIFIED PROTOTYPE"
- board text added: "V2"

Commit message: Hardware: v2 fixes from the two independent reviews
Stop the build on isolation errors and on any rule that does not fire,
on the board and on the panel. Stop the creepage rule reporting rule
areas and mouse bites. Count J2's tabs, copper with no net, in
measure.py. Add XIAO insertion marks to the silkscreen and the assembly
steps to REPORT.md. Copper, BOM and CPL are unchanged.

Co-Authored-By: Claude Opus 5.5 <noreply@anthropic.com>
Other:
- board text added: "5V"
- board text added: "GND"
- board text added: "USB"
